File: USB_voltage_spec.kicad_pcb (KiCad board)
At the start: 2 copper layers, 48.4 x 24.2 mm, 34 parts, among them P1 USB_A, P2 USB_A, P3 USB_OTG, Q1 2N7002, Q2 2N7002, U1 LM4562

Commit message: I lied.
Parts:
- added C5: 100n, Capacitors_SMD:C_0805, B.Cu at (159.6, 56.8)
- moved 2V5 TEST 5.87 mm to (177.1, 48.5), turned to 180 degrees
- moved REF** 2.87 mm to (175.5, 54.0)
- moved R18 0.62 mm to (172.0, 66.0)
- moved R4 0.62 mm to (174.6, 66.0)
- moved R8 0.62 mm to (177.2, 66.0)
- moved Q2 0.62 mm to (171.0, 62.6)
- moved Q1 0.58 mm to (176.2, 62.6)
Connections:
- P2 pad 5: Net-(P2-Pad5) -> Net-(P1-Pad5)
- P3 pad 6: Net-(P3-Pad6) -> Net-(P1-Pad5)
Routing:
- net Net-(P1-Pad5): track 15.0 -> 85.1 mm
- net Net-(P2-Pad5): track 21.9 -> 0.00 mm
- net Net-(P3-Pad6): track 11.2 -> 0.00 mm
- net +5V: track 118.0 -> 113.3 mm
- net Net-(Q1-Pad1): track 25.0 -> 29.5 mm
- net GND: track 13.2 -> 16.6 mm, vias 4 -> 3
- net 2V5_VREF: track 41.7 -> 42.8 mm
- net Net-(D2-Pad2): track 1.39 -> 2.41 mm
- net Net-(D4-Pad2): track 1.39 -> 2.40 mm
- net Net-(D1-Pad2): track 1.39 -> 2.40 mm
- net Net-(Q2-Pad1): track 23.8 -> 24.4 mm
- net USB_D-: track 45.1 -> 44.5 mm
Other:
- rule pad_to_mask_clearance: 0.2 -> 0.19
- board text added: "Board rev: 02"
- board text added: "CC BY-SA 4.0"
- board text removed: "CC BY-SA"
